File: circuit/cellule_orage.sch (KiCad schematic (older format))
At the start: 65 parts, among them Q1 BSS138, Q2 BSS138, Q3 BSS138, SW1 OFF/ON, U2 TLC274, U4 LM555N, U5 TLP291

Commit message: Power update
Added some component to get a proper alimentation
Parts:
- removed P?: Batt+, symbol CONN_01X01
- removed P?: Batt-, symbol CONN_01X01
- removed R19: 38.3k, symbol R_Small
- removed SW1: OFF/ON, symbol SPST
- R?: value 10k -> 140k
- R?: value 10k -> 100k
Connections:
- net GND: no longer U?.1 (/SHDN)
- net Timer_out: no longer P?.5 (P5), Q1.1 (G), Q2.1 (G), Q3.1 (G)
- net LBO: now reaches U?.4 (LBO)
- net BUZZER_OUT renamed buzzer_out
- net Batt+ renamed Vbat
- net Vbat: no longer C6.1, L1.1, R?.2
- net LED_OUT renamed led_out
- net TRIG_OUT renamed trig_out
- new net power_out: C6.1, L1.1, R?.2
- new net timer_out: P?.5 (P5), Q1.1 (G), Q2.1 (G), Q3.1 (G)
Other:
- note added: "Circuit enable"
- note added: "Max 150 [mA]"
- note added: "Max 500 [mA]"
- note added: "Power switch"
- note removed: "Modifier LBI LBO"
- note removed: "POWER ON/OFF"
- moved on the sheet: C10, C12, C6, C7, C8, D1, L1, R14, R15, R?, U?
